Commit message: Add joint number parameters

File: ros2_description_bolt/urdf/bolt/ros2_control/system_bolt.ros2_control.xacro (robot description, xacro)
@@ -20,16 +20,10 @@
             <param name="example_param_hw_stop_duration_sec">3.0</param>
             <param name="example_param_hw_slowdown">${slowdown}</param>
-            <param name="FLHAA">0</param>
-            <param name="FLHFE">1</param>
-            <param name="FLK">2</param>
-            <param name="FRHAA">3</param>
-            <param name="FRHFE">4</param>
-            <param name="FRK">5</param>
-          </xacro:unless>
+            </xacro:unless>
         </hardware>
       </xacro:unless>
       <joint name="FLHAA">
         <command_interface name="position">
-          <param name="min">-0.2</param>
+          <param name="min">-0.5</param>
           <param name="max">0.5</param>
         </command_interface>
@@ -45,9 +39,28 @@
         <state_interface name="velocity"/>
         <state_interface name="acceleration"/>
+        <param name="motor_number">0</param>
       </joint>
       <joint name="FLHFE">
         <command_interface name="position">
+          <param name="min">-1.7</param>
+          <param name="max">1.7</param>
+        </command_interface>
+        <command_interface name="velocity">
           <param name="min">-1</param>
           <param name="max">1</param>
+        </command_interface>
+        <command_interface name="acceleration">
+          <param name="min">-1</param>
+          <param name="max">1</param>
+        </command_interface>
+        <state_interface name="position"/>
+        <state_interface name="velocity"/>
+        <state_interface name="acceleration"/>*
+        <param name="motor_number">1</param>
+      </joint>
+      <joint name="FLK">
+        <command_interface name="position">
+          <param name="min">-3.4</param>
+          <param name="max">3.4</param>
         </command_interface>
         <command_interface name="velocity">
@@ -62,9 +75,10 @@
         <state_interface name="velocity"/>
         <state_interface name="acceleration"/>
+        <param name="motor_number">2</param>
       </joint>
-      <joint name="FLK">
+      <joint name="FRHAA">
         <command_interface name="position">
-          <param name="min">-1.5</param>
-          <param name="max">1.5</param>
+          <param name="min">-0.5</param>
+          <param name="max">0.5</param>
         </command_interface>
         <command_interface name="velocity">
@@ -79,9 +93,10 @@
         <state_interface name="velocity"/>
         <state_interface name="acceleration"/>
+        <param name="motor_number">3</param>
       </joint>
-      <joint name="FRHAA">
+      <joint name="FRHFE">
         <command_interface name="position">
-          <param name="min">-0.5</param>
-          <param name="max">0.2</param>
+          <param name="min">-1.7</param>
+          <param name="max">1.7</param>
         </command_interface>
         <command_interface name="velocity">
@@ -96,26 +111,10 @@
         <state_interface name="velocity"/>
         <state_interface name="acceleration"/>
-      </joint>
-      <joint name="FRHFE">
-        <command_interface name="position">
-          <param name="min">-1</param>
-          <param name="max">1</param>
-        </command_interface>
-        <command_interface name="velocity">
-          <param name="min">-1</param>
-          <param name="max">1</param>
-        </command_interface>
-        <command_interface name="acceleration">
-          <param name="min">-1</param>
-          <param name="max">1</param>
-        </command_interface>
-        <state_interface name="position"/>
-        <state_interface name="velocity"/>
-        <state_interface name="acceleration"/>
+        <param name="motor_number">4</param>
       </joint>
       <joint name="FRK">
         <command_interface name="position">
-          <param name="min">-1.5</param>
-          <param name="max">1.5</param>
+          <param name="min">-3.4</param>
+          <param name="max">3.4</param>
         </command_interface>
         <command_interface name="velocity">
@@ -125,4 +124,5 @@
         <state_interface name="velocity"/>
         <state_interface name="acceleration"/>
+        <param name="motor_number">5</param>
       </joint>
     </ros2_control>
