Commit message: URDF doc for tests on rviz2

File: ros2_description_bolt/urdf/system_bolt.urdf.xacro (robot description, xacro)
@@ -1,24 +1,25 @@
-<!-- Adapted from bolt.urdf.xacro of ODRI (robot_properties_bolt) https://github.com/open-dynamic-robot-initiative/robot_properties_bolt/blob/master/src/robot_properties_bolt/resources/xacro/bolt.urdf.xacro -->
-<?xml version="1.0" ?>
-<robot name="bolt"
-  xmlns:controller="http://playerstage.sourceforge.net/gazebo/xmlschema/#controller"
-  xmlns:interface="http://playerstage.sourceforge.net/gazebo/xmlschema/#interface"
-  xmlns:sensor="http://playerstage.sourceforge.net/gazebo/xmlschema/#sensor"
-  xmlns:xacro="http://playerstage.sourceforge.net/gazebo/xmlschema/#interface">
-  <xacro:property name="mesh_ext" value="stl" />
-  <xacro:property name="color_name" value="grey" />
-  <xacro:property name="color" value="0.8 0.8 0.8" />
-  <xacro:property name="opacity" value="1.0" />
-  <xacro:property name="new_leg" value="true" />
-  <xacro:property name="has_passive_ankle" value="false" />
-  <!-- Include the legs -->
-  <xacro:include filename="bolt.xacro"/>
-  <!-- Include the fully parametrized bolt -->
-  <xacro:bolt_full
-      mesh_ext="${mesh_ext}"
-      color_name="${color_name}"
-      color="${color}"
-      opacity="${opacity}"
-      new_leg="${new_leg}"
-      has_passive_ankle="${has_passive_ankle}"/>
+<?xml version="1.0"?>
+<!-- Revolute-Revolute Manipulator -->
+<!--
+Copied and modified from ROS2 example -
+https://github.com/ros-controls/ros2_control_demos/blob/master/ros2_control_demo_description/rrbot_description/urdf/rrbot.urdf.xacro
+-->
+<robot xmlns:xacro="http://www.ros.org/wiki/xacro" name="bolt">
+  <xacro:arg name="prefix" default="" />
+  <!-- Import RRBot macro -->
+  <xacro:include filename="$(find ros2_description_bolt)/urdf/system_bolt_description.urdf.xacro" />
+  <!-- Import Rviz colors -->
+  <xacro:include filename="$(find ros2_description_bolt)/gazebo/system_bolt.materials.xacro" />
+  <!-- Import RRBot ros2_control description -->
+  <xacro:include filename="$(find ros2_description_bolt)/ros2_control/system_bolt.ros2_control.xacro" />
+  <!-- Used for fixing robot -->
+  <link name="world"/>
+  <gazebo reference="world">
+    <static>true</static>
+  </gazebo>
+  <xacro:system_bolt parent="world" prefix="$(arg prefix)">
+    <origin xyz="0 0 0" rpy="0 0 0" />
+  </xacro:system_bolt>
+  <xacro:system_bolt_ros2_control
+    name="Bolt" prefix="$(arg prefix)" />
 </robot>
