Commit message: Ajout du controleur gazebo_ros2_bolt avec les modifications requises

File: ros2_description_bolt/urdf/system_bolt_description.urdf.xacro (robot description, xacro)
@@ -14,6 +14,7 @@
   <xacro:property name="opacity" value="1.0" />
   <xacro:property name="new_leg" value="true" />
-  <xacro:property name="has_passive_ankle" value="false" />
+  <xacro:property name="has_passive_ankle" value="true" />
   <xacro:arg name="prefix" default="" />
+  <xacro:arg name="use_crane" default="false" />
   <xacro:arg name="use_sim" default="false" />
   <xacro:arg name="use_fake_hardware" default="false" />
@@ -27,9 +28,9 @@
   <!-- ros_control plugin -->
   <gazebo>
-    <plugin name="gazebo_ros2_control" filename="libgazebo_ros2_control.so">
+    <plugin name="gazebo_ros2_bolt" filename="libgazebo_ros2_control.so">
       <parameters>$(find ros2_control_bolt_bringup)/config/bolt_gazebo_forward_controller_position.yaml</parameters>
     </plugin>
   </gazebo>
-  <xacro:if value="$(arg use_sim)">
+  <xacro:if value="$(arg use_crane)">
      <xacro:crane parent="base_link" />
   </xacro:if>
