Commit message: Modif step by step

File: ros2_description_bolt/ros2_control/system_bolt.ros2_control.xacro (robot description, xacro)
@@ -1,5 +1,5 @@
 <?xml version="1.0"?>
 <robot xmlns:xacro="http://www.ros.org/wiki/xacro">
-  <xacro:macro name="system_bolt" params="name prefix use_sim:=^|false use_fake_hardware:=^|true fake_sensor_commands:=^|false slowdown:=2.0">
+  <xacro:macro name="system_bolt_ros2_control" params="name prefix use_sim:=^|false use_fake_hardware:=^|true fake_sensor_commands:=^|false slowdown:=2.0">
     <ros2_control name="${name}" type="system">
       <xacro:if value="$(arg use_sim)">

File: ros2_description_bolt/urdf/system_bolt.urdf.xacro (robot description, xacro)
@@ -1,25 +1,77 @@
-<?xml version="1.0"?>
-<!-- Revolute-Revolute Manipulator -->
+<?xml version="1.0" ?>
 <!--
-Copied and modified from ROS2 example -
-https://github.com/ros-controls/ros2_control_demos/blob/master/ros2_control_demo_description/rrbot_description/urdf/rrbot.urdf.xacro
+Copied from ODRI -
+https://github.com/open-dynamic-robot-initiative/robot_properties_bolt/blob/master/src/robot_properties_bolt/resources/xacro/bolt.xacro
 -->
-<robot xmlns:xacro="http://www.ros.org/wiki/xacro" name="bolt">
-  <xacro:arg name="prefix" default="" />
-  <!-- Import RRBot macro -->
-  <xacro:include filename="$(find ros2_description_bolt)/urdf/system_bolt_description.urdf.xacro" />
-  <!-- Import Rviz colors -->
-  <xacro:include filename="$(find ros2_description_bolt)/gazebo/system_bolt.materials.xacro" />
-  <!-- Import RRBot ros2_control description -->
-  <xacro:include filename="$(find ros2_description_bolt)/ros2_control/system_bolt.ros2_control.xacro" />
-  <!-- Used for fixing robot -->
-  <link name="world"/>
-  <gazebo reference="world">
-    <static>true</static>
-  </gazebo>
-  <xacro:system_bolt parent="world" prefix="$(arg prefix)">
-    <origin xyz="0 0 0" rpy="0 0 0" />
-  </xacro:system_bolt>
-  <xacro:system_bolt_ros2_control
-    name="Bolt" prefix="$(arg prefix)" />
+<robot name="bolt"
+  xmlns:controller="http://playerstage.sourceforge.net/gazebo/xmlschema/#controller"
+  xmlns:interface="http://playerstage.sourceforge.net/gazebo/xmlschema/#interface"
+  xmlns:sensor="http://playerstage.sourceforge.net/gazebo/xmlschema/#sensor"
+  xmlns:xacro="http://playerstage.sourceforge.net/gazebo/xmlschema/#interface">
+  <xacro:macro name="bolt_full" params="mesh_ext color_name color opacity new_leg has_passive_ankle">
+    <!-- This file is based on: https://atlas.is.localnet/confluence/display/AMDW/Quadruped+URDF+Files -->
+    <link name="base_link">
+      <!-- BASE LINK INERTIAL -->
+      <inertial>
+          <origin xyz="0 0 0" rpy="0 0 0" />
+          <mass value="0.61436936"/>
+          <!-- The base is extremely symmetrical. -->
+          <inertia ixx="0.00578574" ixy="0.0" ixz="0.0"
+                                    iyy="0.01938108" iyz="0.0"
+                                                    izz="0.02476124"
+          />
+      </inertial>
+      <!-- BASE LINK VISUAL -->
+      <visual>
+          <origin xyz="0 0 0" rpy="0 0 0" />
+          <geometry>
+            <mesh filename="package://ros2_description_bolt/meshes/${mesh_ext}/bolt_body.${mesh_ext}"/>
+          </geometry>
+          <material name="${color_name}">
+              <color rgba="${color} ${opacity}"/>
+          </material>
+      </visual>
+      <!-- BASE LINK COLLISION -->
+      <collision>
+          <origin xyz="0 0 0" rpy="0 0 0" />
+          <geometry>
+            <mesh filename="package://ros2_description_bolt/meshes/${mesh_ext}/bolt_body.${mesh_ext}"/>
+          </geometry>
+          <material name="${color_name}">
+              <color rgba="${color} ${opacity}"/>
+          </material>
+      </collision>
+      <!-- Bullet specific paramters -->
+      <contact>
+        <lateral_friction value="1.0"/>
+        <restitution value="0.5"/>
+      </contact>
+    </link> <!-- END BASE LINK -->
+    <!-- Include the legs -->
+    <xacro:include filename="leg.xacro"/>
+    <!-- Include the front left leg -->
+    <xacro:leg
+        prefix="FL"
+        is_front="true"
+        is_right="false"
+        has_side_motion="true"
+        mesh_ext="${mesh_ext}"
+        color_name="${color_name}"
+        color="${color}"
+        opacity="${opacity}"
+        new_leg="${new_leg}"
+        has_passive_ankle="${has_passive_ankle}"/>
+    <!-- Include the front right leg -->
+    <xacro:leg
+        prefix="FR"
+        is_front="true"
+        is_right="true"
+        has_side_motion="true"
+        mesh_ext="${mesh_ext}"
+        color_name="${color_name}"
+        color="${color}"
+        opacity="${opacity}"
+        new_leg="${new_leg}"
+        has_passive_ankle="${has_passive_ankle}"/>
+  </xacro:macro>
 </robot>

File: ros2_description_bolt/urdf/system_bolt_description.urdf.xacro (robot description, xacro)
@@ -1,7 +1,7 @@
+<?xml version="1.0" ?>
 <!--
 Copied from ODRI -
 https://github.com/open-dynamic-robot-initiative/robot_properties_bolt/blob/master/src/robot_properties_bolt/resources/xacro/bolt.urdf.xacro
 -->
-<?xml version="1.0" ?>
 <robot name="bolt"
   xmlns:controller="http://playerstage.sourceforge.net/gazebo/xmlschema/#controller"
@@ -15,6 +15,10 @@
   <xacro:property name="new_leg" value="true" />
   <xacro:property name="has_passive_ankle" value="false" />
+  <xacro:arg name="prefix" default="" />
+  <xacro:arg name="use_sim" default="false" />
+  <xacro:arg name="use_fake_hardware" default="false" />
   <!-- Include the legs -->
-  <xacro:include filename="system_bolt.xacro"/>
+  <xacro:include filename="system_bolt.urdf.xacro"/>
+  <xacro:include filename="$(find ros2_description_bolt)/ros2_control/system_bolt.ros2_control.xacro" />
   <!-- Include the fully parametrized bolt -->
   <xacro:bolt_full
@@ -25,3 +29,5 @@
       new_leg="${new_leg}"
       has_passive_ankle="${has_passive_ankle}"/>
+  <xacro:system_bolt_ros2_control
+    name="SystemBoltRos2Control" prefix="$(arg prefix)" use_fake_hardware="$(arg use_fake_hardware)"/>
 </robot>

Commit message: Changes about compilation fails

File: ros2_description_bolt/ros2_control/system_bolt.ros2_control.xacro (robot description, xacro)
@@ -1,5 +1,5 @@
 <?xml version="1.0"?>
 <robot xmlns:xacro="http://www.ros.org/wiki/xacro">
-  <xacro:macro name="system_bolt_ros2_control" params="name prefix use_sim:=^|false use_fake_hardware:=^|true fake_sensor_commands:=^|false slowdown:=2.0">
+  <xacro:macro name="system_bolt_ros2_control" params="name prefix use_sim:=^|false use_fake_hardware:=^|true fake_sensor_commands:=^|false slowdown:=2.0 enp3s0:=^|enp3s0 true:=^|true false:=^|false">
     <ros2_control name="${name}" type="system">
       <xacro:if value="$(arg use_sim)">

File: ros2_description_bolt/urdf/leg.xacro (robot description, xacro)
@@ -1,5 +1,5 @@
 <?xml version="1.0"?>
 <robot xmlns:xacro="http://playerstage.sourceforge.net/gazebo/xmlschema/#interface" name="bolt">
-<!-- See TODO: add the wiki link here -->
+<!-- See TODO add the wiki link here -->
 <!-- These are absolute distance value, the sign are decided below -->
     <xacro:property name="base_2_HAA_x" value="${0.0 * 0.001}" />
@@ -47,5 +47,5 @@
         </joint>
         <link name="${prefix}_SHOULDER">
-        <!-- TODO: Update inertias and add visuals for link. -->
+        <!-- TODO Update inertias and add visuals for link. -->
         <!-- create a dummy shoulder link to join the two joints -->
             <inertial>
@@ -210,5 +210,5 @@
         </link>
         <!-- END UPPER LEG LINK -->
-        <!-- KFE: Joint between the upper leg and the lower leg -->
+        <!-- KFE Joint between the upper leg and the lower leg -->
         <joint name="${prefix}_KFE" type="revolute">
             <parent link="${prefix}_UPPER_LEG"/>
@@ -312,5 +312,5 @@
         </link>
         <!-- END LOWER LEG LINK -->
-        <!-- KFE: Joint between the upper leg and the lower leg -->
+        <!-- KFE Joint between the upper leg and the lower leg -->
         <joint name="${prefix}_ANKLE" type="${ankle_joint_type}">
             <parent link="${prefix}_LOWER_LEG"/>

File: ros2_description_bolt/urdf/system_bolt.urdf.xacro (robot description, xacro)
@@ -10,5 +10,5 @@
   xmlns:xacro="http://playerstage.sourceforge.net/gazebo/xmlschema/#interface">
   <xacro:macro name="bolt_full" params="mesh_ext color_name color opacity new_leg has_passive_ankle">
-    <!-- This file is based on: https://atlas.is.localnet/confluence/display/AMDW/Quadruped+URDF+Files -->
+    <!-- This file is based on https://atlas.is.localnet/confluence/display/AMDW/Quadruped+URDF+Files -->
     <link name="base_link">
       <!-- BASE LINK INERTIAL -->
